Commit message: update model to V2

File: premaidai_gym/models_robot/premaidai_description/urdf/premaidai.urdf (robot description, URDF)
Before this commit: robot premaidai, 27 links, 26 joints
Links:
- removed link head_dummy
- removed link l_dummy
- removed link neck
- removed link r_dummy
- added link head_yaw, mass 0.01; collision mesh filename=package://premaidai_description/meshes/neck_yaw.dae; visual mesh filename=package://premaidai_description/meshes/neck_yaw.dae
- added link l_ankle, mass 0.01; collision mesh filename=package://premaidai_description/meshes/l_ankle.dae; visual mesh filename=package://premaidai_description/meshes/l_ankle.dae
- added link neck_pitch, mass 0.01; collision mesh filename=package://premaidai_description/meshes/neck_pitch.dae; visual mesh filename=package://premaidai_description/meshes/neck_pitch.dae
- added link r_ankle, mass 0.01; collision mesh filename=package://premaidai_description/meshes/r_ankle.dae; visual mesh filename=package://premaidai_description/meshes/r_ankle.dae
- link base_link: mass None -> 0.001
Joints:
- joint body_to_base_link: origin xyz=0.0236 0 0 rpy=0 0 0 -> xyz=0 0 0 rpy=0 0 0
- joint head_nx_joint: origin xyz=0 0 0.0362 rpy=0 0 0 -> xyz=0 0 0.0129 rpy=0 0 0; parent head_dummy -> head_yaw
- joint head_ny_joint: child neck -> neck_pitch; origin xyz=-0.0319 0 0.1088 rpy=0 0 0 -> xyz=0.0038738 0 0.132809 rpy=0 0 0
- joint head_nz_joint: child head_dummy -> head_yaw; origin xyz=0 0 0 rpy=0 0 0 -> xyz=-0.0103485 0 0.011103 rpy=0 0 0; parent neck -> neck_pitch
- joint l_akx_joint: limit lower=-1.5707963268 upper=1.5707963268 effort=0 velocity=0 -> lower=-0.650898727916 upper=0.667392089347 effort=0 velocity=0; origin (none) -> xyz=0 0 -0.040677 rpy=0 0 0; parent l_dummy -> l_ankle
- joint l_aky_joint: child l_dummy -> l_ankle; limit lower=-1.5707963268 upper=1.5707963268 effort=0 velocity=0 -> lower=-1.07089039579 upper=0.424115008235 effort=0 velocity=0; origin xyz=0 0 -0.06749 rpy=0 0 0 -> xyz=0 0 -0.065 rpy=0 0 0
- joint l_elx_joint: limit lower=-1.5707963268 upper=1.5707963268 effort=0 velocity=0 -> lower=-2.07639639448 upper=0.235619449019 effort=0 velocity=0; origin xyz=0 0.0304889766965 0 rpy=0 0 0 -> xyz=0 0.024054 0 rpy=0 0 0
- joint l_ely_joint: limit lower=-1.5707963268 upper=1.5707963268 effort=0 velocity=0 -> lower=-2.24604239778 upper=2.34441351774 effort=0 velocity=0; origin xyz=0 0.05587567 0 rpy=0 0 0 -> xyz=0.0088013 0.060007 0 rpy=0 0 0
- joint l_hpx_joint: limit lower=-1.5707963268 upper=1.5707963268 effort=0 velocity=0 -> lower=-0.396416633005 upper=0.442440965381 effort=0 velocity=0; origin xyz=0 0 -0.05407 rpy=0 0 0 -> xyz=0 -0.0021 -0.028 rpy=0 0 0
- joint l_hpy_joint: limit lower=-1.5707963268 upper=1.5707963268 effort=0 velocity=0 -> lower=-1.59872159483 upper=1.5745138781 effort=0 velocity=0; origin xyz=0 0.01021 -0.03829 rpy=0 0 0 -> xyz=0 0.0128525 -0.034358 rpy=0 0 0
- joint l_hpz_joint: limit lower=-1.5707963268 upper=1.5707963268 effort=0 velocity=0 -> lower=-1.41371669412 upper=1.78774075282 effort=0 velocity=0; origin xyz=0 0.0217 0.01505 rpy=0 0 0 -> xyz=0.004225 0.0195245 0.001412 rpy=0 0 0
- joint l_kny_joint: limit lower=-1.5707963268 upper=1.5707963268 effort=0 velocity=0 -> lower=-0.036521014598 upper=2.08811191709 effort=0 velocity=0; origin xyz=0 0 -0.06827 rpy=0 0 0 -> xyz=0 0 -0.0652 rpy=0 0 0
- joint l_shx_joint: limit lower=-1.5707963268 upper=1.5707963268 effort=0 velocity=0 -> lower=-1.59808891297 upper=0.0530143760293 effort=0 velocity=0; origin xyz=0 0.01925 0 rpy=0 0 0 -> xyz=0 0.0189 0 rpy=0 0 0
- joint l_shy_joint: limit lower=-1.5707963268 upper=1.5707963268 effort=0 velocity=0 -> lower=-1.88495559215 upper=2.23838476568 effort=0 velocity=0; origin xyz=-0.01726 0.03829 0.097 rpy=0 0 0 -> xyz=0 0.0359 0.113043 rpy=0 0 0
- joint l_wry_joint: limit lower=-1.5707963268 upper=1.5707963268 effort=0 velocity=0 -> lower=-2.35619449019 upper=2.06167017892 effort=0 velocity=0; origin xyz=0.01002 0.0476117842556 0 rpy=0 0 0 -> xyz=0 0.061348 0 rpy=0 0 0
- joint r_akx_joint: limit lower=-1.5707963268 upper=1.5707963268 effort=0 velocity=0 -> lower=-0.667392089347 upper=0.650898727916 effort=0 velocity=0; origin (none) -> xyz=0 0 -0.040677 rpy=0 0 0; parent r_dummy -> r_ankle
- joint r_aky_joint: child r_dummy -> r_ankle; limit lower=-1.5707963268 upper=1.5707963268 effort=0 velocity=0 -> lower=-1.07089039579 upper=0.424115008235 effort=0 velocity=0; origin xyz=0 0 -0.06749 rpy=0 0 0 -> xyz=0 0 -0.065 rpy=0 0 0
- joint r_elx_joint: limit lower=-1.5707963268 upper=1.5707963268 effort=0 velocity=0 -> lower=-0.235619449019 upper=2.07639639448 effort=0 velocity=0; origin xyz=0 -0.0304889766965 0 rpy=0 0 0 -> xyz=0 -0.024054 0 rpy=0 0 0
- joint r_ely_joint: limit lower=-1.5707963268 upper=1.5707963268 effort=0 velocity=0 -> lower=-2.24604239778 upper=2.34441351774 effort=0 velocity=0; origin xyz=0 -0.05587567 0 rpy=0 0 0 -> xyz=0.0088013 -0.060007 0 rpy=0 0 0
- joint r_hpx_joint: limit lower=-1.5707963268 upper=1.5707963268 effort=0 velocity=0 -> lower=-0.442440965381 upper=0.396416633005 effort=0 velocity=0; origin xyz=0 0 -0.05407 rpy=0 0 0 -> xyz=0 0.0021 -0.028 rpy=0 0 0
- joint r_hpy_joint: limit lower=-1.5707963268 upper=1.5707963268 effort=0 velocity=0 -> lower=-1.59872159483 upper=1.5745138781 effort=0 velocity=0; origin xyz=0 -0.01021 -0.03829 rpy=0 0 0 -> xyz=0 -0.0128525 -0.034358 rpy=0 0 0
- joint r_hpz_joint: limit lower=-1.5707963268 upper=1.5707963268 effort=0 velocity=0 -> lower=-1.41371669412 upper=1.78774075282 effort=0 velocity=0; origin xyz=0 -0.0217 0.01505 rpy=0 0 0 -> xyz=0.004225 -0.0195245 0.001412 rpy=0 0 0
- joint r_kny_joint: limit lower=-1.5707963268 upper=1.5707963268 effort=0 velocity=0 -> lower=-0.036521014598 upper=2.08811191709 effort=0 velocity=0; origin xyz=0 0 -0.06827 rpy=0 0 0 -> xyz=0 0 -0.0652 rpy=0 0 0
- joint r_shx_joint: limit lower=-1.5707963268 upper=1.5707963268 effort=0 velocity=0 -> lower=-0.0530143760293 upper=1.59808891297 effort=0 velocity=0; origin xyz=0 -0.01925 0 rpy=0 0 0 -> xyz=0 -0.0189 0 rpy=0 0 0
- joint r_shy_joint: limit lower=-1.5707963268 upper=1.5707963268 effort=0 velocity=0 -> lower=-1.88495559215 upper=2.23838476568 effort=0 velocity=0; origin xyz=-0.01726 -0.03829 0.097 rpy=0 0 0 -> xyz=0 -0.0359 0.113043 rpy=0 0 0
- joint r_wry_joint: limit lower=-1.5707963268 upper=1.5707963268 effort=0 velocity=0 -> lower=-2.35619449019 upper=2.06167017892 effort=0 velocity=0; origin xyz=0.01002 -0.0476117842556 0 rpy=0 0 0 -> xyz=0 -0.061348 0 rpy=0 0 0

Commit message: apply proper inertia data from chikuta-san's urdf

File: premaidai_gym/models_robot/premaidai_description/urdf/premaidai.urdf (robot description, URDF)
Before this commit: robot premaidai, 27 links, 26 joints
Links:
- link body: mass 0.01 -> 0.4426
- link head: mass 0.01 -> 0.1449
- link l_ankle: mass 0.01 -> 0.0571
- link l_foot: mass 0.01 -> 0.0941
- link l_hand: mass 0.01 -> 0.0046
- link l_hip_joint: mass 0.01 -> 0.0143
- link l_larm: mass 0.01 -> 0.0812
- link l_larm_joint: mass 0.01 -> 0.0124
- link l_lleg: mass 0.01 -> 0.0719
- link l_uarm: mass 0.01 -> 0.0712
- link l_uarm_joint: mass 0.01 -> 0.0131
- link l_uleg: mass 0.01 -> 0.1134
- link l_uleg_root: mass 0.01 -> 0.0648
- link r_ankle: mass 0.01 -> 0.0571
- link r_foot: mass 0.01 -> 0.0941
- link r_hand: mass 0.01 -> 0.0046
- link r_hip_joint: mass 0.01 -> 0.0143
- link r_larm: mass 0.01 -> 0.0812
- link r_larm_joint: mass 0.01 -> 0.0124
- link r_lleg: mass 0.01 -> 0.0719
- link r_uarm: mass 0.01 -> 0.0712
- link r_uarm_joint: mass 0.01 -> 0.0131
- link r_uleg: mass 0.01 -> 0.1134
- link r_uleg_root: mass 0.01 -> 0.0648
