Commit message: shorten urdf load path
urdf loader couldn't load the path longer than 128.

File: premaidai_gym/assets/premaidai.urdf (robot description, URDF)
Before this commit: robot premaidai, 27 links, 26 joints
Links:
- link body: geometry collision mesh filename=package://assets/meshes/body.dae; visual mesh filename=package://assets/meshes/body.dae
- link head: geometry collision mesh filename=package://assets/meshes/head.dae; visual mesh filename=package://assets/meshes/head.dae
- link head_yaw: geometry collision mesh filename=package://assets/meshes/neck_yaw.dae; visual mesh filename=package://assets/meshes/neck_yaw.dae
- link l_ankle: geometry collision mesh filename=package://assets/meshes/l_ankle.dae; visual mesh filename=package://assets/meshes/l_ankle.dae
- link l_foot: geometry collision mesh filename=package://assets/meshes/l_foot.dae; visual mesh filename=package://assets/meshes/l_foot.dae
- link l_hand: geometry collision mesh filename=package://assets/meshes/l_hand.dae; visual mesh filename=package://assets/meshes/l_hand.dae
- link l_hip_joint: geometry collision mesh filename=package://assets/meshes/l_hip_joint.dae; visual mesh filename=package://assets/meshes/l_hip_joint.dae
- link l_larm: geometry collision mesh filename=package://assets/meshes/l_larm.dae; visual mesh filename=package://assets/meshes/l_larm.dae
- link l_larm_joint: geometry collision mesh filename=package://assets/meshes/l_larm_joint.dae; visual mesh filename=package://assets/meshes/l_larm_joint.dae
- link l_lleg: geometry collision mesh filename=package://assets/meshes/l_lleg.dae; visual mesh filename=package://assets/meshes/l_lleg.dae
- link l_uarm: geometry collision mesh filename=package://assets/meshes/l_uarm.dae; visual mesh filename=package://assets/meshes/l_uarm.dae
- link l_uarm_joint: geometry collision mesh filename=package://assets/meshes/l_uarm_joint.dae; visual mesh filename=package://assets/meshes/l_uarm_joint.dae
- link l_uleg: geometry collision mesh filename=package://assets/meshes/l_uleg.dae; visual mesh filename=package://assets/meshes/l_uleg.dae
- link l_uleg_root: geometry collision mesh filename=package://assets/meshes/l_uleg_root.dae; visual mesh filename=package://assets/meshes/l_uleg_root.dae
- link neck_pitch: geometry collision mesh filename=package://assets/meshes/neck_pitch.dae; visual mesh filename=package://assets/meshes/neck_pitch.dae
- link r_ankle: geometry collision mesh filename=package://assets/meshes/r_ankle.dae; visual mesh filename=package://assets/meshes/r_ankle.dae
- link r_foot: geometry collision mesh filename=package://assets/meshes/r_foot.dae; visual mesh filename=package://assets/meshes/r_foot.dae
- link r_hand: geometry collision mesh filename=package://assets/meshes/r_hand.dae; visual mesh filename=package://assets/meshes/r_hand.dae
- link r_hip_joint: geometry collision mesh filename=package://assets/meshes/r_hip_joint.dae; visual mesh filename=package://assets/meshes/r_hip_joint.dae
- link r_larm: geometry collision mesh filename=package://assets/meshes/r_larm.dae; visual mesh filename=package://assets/meshes/r_larm.dae
- link r_larm_joint: geometry collision mesh filename=package://assets/meshes/r_larm_joint.dae; visual mesh filename=package://assets/meshes/r_larm_joint.dae
- link r_lleg: geometry collision mesh filename=package://assets/meshes/r_lleg.dae; visual mesh filename=package://assets/meshes/r_lleg.dae
- link r_uarm: geometry collision mesh filename=package://assets/meshes/r_uarm.dae; visual mesh filename=package://assets/meshes/r_uarm.dae
- link r_uarm_joint: geometry collision mesh filename=package://assets/meshes/r_uarm_joint.dae; visual mesh filename=package://assets/meshes/r_uarm_joint.dae
- link r_uleg: geometry collision mesh filename=package://assets/meshes/r_uleg.dae; visual mesh filename=package://assets/meshes/r_uleg.dae
- link r_uleg_root: geometry collision mesh filename=package://assets/meshes/r_uleg_root.dae; visual mesh filename=package://assets/meshes/r_uleg_root.dae

Commit message: add joint speed limit information to urdf

File: premaidai_gym/assets/premaidai.urdf (robot description, URDF)
Before this commit: robot premaidai, 27 links, 26 joints
Joints:
- joint head_nx_joint: limit lower=-0.382881604656 upper=0.500691329166 effort=0 velocity=0 -> lower=-0.382881604656 upper=0.500691329166 effort=0 velocity=428.6
- joint head_ny_joint: limit lower=-0.176714586764 upper=0.412334035784 effort=0 velocity=0 -> lower=-0.176714586764 upper=0.412334035784 effort=0 velocity=428.6
- joint head_nz_joint: limit lower=-0.824668071567 upper=0.824668071567 effort=0 velocity=0 -> lower=-0.824668071567 upper=0.824668071567 effort=0 velocity=428.6
- joint l_akx_joint: limit lower=-0.650898727916 upper=0.667392089347 effort=0 velocity=0 -> lower=-0.650898727916 upper=0.667392089347 effort=0 velocity=428.6
- joint l_aky_joint: limit lower=-1.07089039579 upper=0.424115008235 effort=0 velocity=0 -> lower=-1.07089039579 upper=0.424115008235 effort=0 velocity=428.6
- joint l_elx_joint: limit lower=-2.07639639448 upper=0.235619449019 effort=0 velocity=0 -> lower=-2.07639639448 upper=0.235619449019 effort=0 velocity=428.6
- joint l_ely_joint: limit lower=-2.24604239778 upper=2.34441351774 effort=0 velocity=0 -> lower=-2.24604239778 upper=2.34441351774 effort=0 velocity=428.6
- joint l_hpx_joint: limit lower=-0.396416633005 upper=0.442440965381 effort=0 velocity=0 -> lower=-0.396416633005 upper=0.442440965381 effort=0 velocity=428.6
- joint l_hpy_joint: limit lower=-1.59872159483 upper=1.5745138781 effort=0 velocity=0 -> lower=-1.59872159483 upper=1.5745138781 effort=0 velocity=428.6
- joint l_hpz_joint: limit lower=-1.41371669412 upper=1.78774075282 effort=0 velocity=0 -> lower=-1.41371669412 upper=1.78774075282 effort=0 velocity=428.6
- joint l_kny_joint: limit lower=-0.036521014598 upper=2.08811191709 effort=0 velocity=0 -> lower=-0.036521014598 upper=2.08811191709 effort=0 velocity=428.6
- joint l_shx_joint: limit lower=-1.59808891297 upper=0.0530143760293 effort=0 velocity=0 -> lower=-1.59808891297 upper=0.0530143760293 effort=0 velocity=428.6
- joint l_shy_joint: limit lower=-1.88495559215 upper=2.23838476568 effort=0 velocity=0 -> lower=-1.88495559215 upper=2.23838476568 effort=0 velocity=428.6
- joint l_wry_joint: limit lower=-2.35619449019 upper=2.06167017892 effort=0 velocity=0 -> lower=-2.35619449019 upper=2.06167017892 effort=0 velocity=428.6
- joint r_akx_joint: limit lower=-0.667392089347 upper=0.650898727916 effort=0 velocity=0 -> lower=-0.667392089347 upper=0.650898727916 effort=0 velocity=428.6
- joint r_aky_joint: limit lower=-1.07089039579 upper=0.424115008235 effort=0 velocity=0 -> lower=-1.07089039579 upper=0.424115008235 effort=0 velocity=428.6
- joint r_elx_joint: limit lower=-0.235619449019 upper=2.07639639448 effort=0 velocity=0 -> lower=-0.235619449019 upper=2.07639639448 effort=0 velocity=428.6
- joint r_ely_joint: limit lower=-2.24604239778 upper=2.34441351774 effort=0 velocity=0 -> lower=-2.24604239778 upper=2.34441351774 effort=0 velocity=428.6
- joint r_hpx_joint: limit lower=-0.442440965381 upper=0.396416633005 effort=0 velocity=0 -> lower=-0.442440965381 upper=0.396416633005 effort=0 velocity=428.6
- joint r_hpy_joint: limit lower=-1.59872159483 upper=1.5745138781 effort=0 velocity=0 -> lower=-1.59872159483 upper=1.5745138781 effort=0 velocity=428.6
- joint r_hpz_joint: limit lower=-1.41371669412 upper=1.78774075282 effort=0 velocity=0 -> lower=-1.41371669412 upper=1.78774075282 effort=0 velocity=428.6
- joint r_kny_joint: limit lower=-0.036521014598 upper=2.08811191709 effort=0 velocity=0 -> lower=-0.036521014598 upper=2.08811191709 effort=0 velocity=428.6
- joint r_shx_joint: limit lower=-0.0530143760293 upper=1.59808891297 effort=0 velocity=0 -> lower=-0.0530143760293 upper=1.59808891297 effort=0 velocity=428.6
- joint r_shy_joint: limit lower=-1.88495559215 upper=2.23838476568 effort=0 velocity=0 -> lower=-1.88495559215 upper=2.23838476568 effort=0 velocity=428.6
- joint r_wry_joint: limit lower=-2.35619449019 upper=2.06167017892 effort=0 velocity=0 -> lower=-2.35619449019 upper=2.06167017892 effort=0 velocity=428.6
